File: KDT_Hierarchical_KiBot.kicad_pcb (KiCad board)
At the start: 6 copper layers, 0 parts

Commit message: feat: Changed templates to be specific to Ryan Dynamics
Other:
- board text added: "ALL DIMENSIONS IN MILLIMETERS UNLESS OTHERWISE SPECIFIED."
- board text added: "BOTTOM VIEW"
- board text added: "COMPONENTS"
- board text added: "DRILL TABLE"
- board text added: "IMPEDANCE TABLE"
- board text added: "LAYER STACKUP LEGEND"
- board text added: "TOP VIEW"
- board text removed: "All dimensions are in millimeters unless otherwise specified."
- board text removed: "Bottom View"
- board text removed: "Components"
- board text removed: "Drill Table"
- board text removed: "Impedance Table"
- board text removed: "Layer Stack Legend"
- board text removed: "Top View"
