File: KDT_Hierarchical_KiBot.kicad_sch (KiCad schematic)
At the start: 0 parts

Commit message: feat: Changed templates to be specific to Ryan Dynamics
Other:
- note added: "CHECKED - PCB LAYOUT CHECKED, CONTACT ENGINEER IF MISTAKE FOUND"
- note added: "COMMENT"
- note added: "DRAFT - EARLY STAGE SCHEMATIC CAPTURE"
- note added: "NOT FITTED COMPONENTS MARKED AS"
- note added: "PRELIMINARY - LATE STAGE SCHEMATIC CAPTURE"
- note added: "RELEASED - READY FOR PRODUCTION"
- note added: "REV ${REVISION}"
- note added: "VARIANT: ${VARIANT}"
- note removed: "CHECKED - There shouldn't be any mistakes. Contact the engineer if you find any."
- note removed: "Comment"
- note removed: "DRAFT - Very early stage of schematic, ignore details."
- note removed: "Date: ${RELEASE_DATE}"
- note removed: "Not fitted components are marked as"
- note removed: "PRELIMINARY - Close to final schematic."
- note removed: "RELEASED - A board with this schematic has been sent to production."
- note removed: "Rev ${REVISION}"
- note removed: "Variant: ${VARIANT}"
