File: subschematic-a.kicad_sch (KiCad schematic)
At the start: 4 parts, among them U1 NE555D

Commit message: feat: prepare Boardwright template workflow
Parts:
- removed D1: LED, LED_THT:LED_D5.0mm_FlatTop, symbol Device:LED
- removed R1: R, Resistor_THT:R_Axial_DIN0617_L17.0mm_D6.0mm_P30.48mm_Horizontal, symbol Device:R
- removed TP1: TestPoint, RD-Testpoints:TestPoint_Pad_D1.5mm, symbol Connector:TestPoint
- removed U1: NE555D, Package_SO:SOIC-8_3.9x4.9mm_P1.27mm, symbol Timer:NE555D
Connections:
- no-connect marks 13 -> 1
